Commit message: Replace mecanum wheel collision meshes with cylinders
Mecanum STL collision meshes have angled rollers that cause lateral
drift during rotation with the DiffDrive plugin. Simple cylinder
collisions (r=0.048, l=0.035) give predictable differential drive
behavior. Visual meshes still show mecanum wheels.

File: urdf/jetrover_description/urdf/car_mecanum.urdf.xacro (robot description, xacro)
@@ -62,10 +62,7 @@
     </visual>
     <collision>
-      <origin
-        xyz="0 0 0"
-        rpy="0 0 0" />
-      <geometry>
-        <mesh
-          filename="package://jetrover_description/meshes/mecanum/wheel_left_front_link_collision.stl" />
+      <origin xyz="0 0 0" rpy="1.5708 0 0" />
+      <geometry>
+        <cylinder radius="0.048" length="0.035" />
       </geometry>
     </collision>
@@ -111,10 +108,7 @@
     </visual>
     <collision>
-      <origin
-        xyz="0 0 0"
-        rpy="0 0 0" />
-      <geometry>
-        <mesh
-          filename="package://jetrover_description/meshes/mecanum/wheel_left_back_link_collision.stl" />
+      <origin xyz="0 0 0" rpy="1.5708 0 0" />
+      <geometry>
+        <cylinder radius="0.048" length="0.035" />
       </geometry>
     </collision>
@@ -160,10 +154,7 @@
     </visual>
     <collision>
-      <origin
-        xyz="0 0 0"
-        rpy="0 0 0" />
-      <geometry>
-        <mesh
-            filename="package://jetrover_description/meshes/mecanum/wheel_right_front_link_collision.stl" />
+      <origin xyz="0 0 0" rpy="1.5708 0 0" />
+      <geometry>
+        <cylinder radius="0.048" length="0.035" />
       </geometry>
     </collision>
@@ -209,10 +200,7 @@
     </visual>
     <collision>
-      <origin
-        xyz="0 0 0"
-        rpy="0 0 0" />
-      <geometry>
-        <mesh
-            filename="package://jetrover_description/meshes/mecanum/wheel_right_back_link_collision.stl" />
+      <origin xyz="0 0 0" rpy="1.5708 0 0" />
+      <geometry>
+        <cylinder radius="0.048" length="0.035" />
       </geometry>
     </collision>
