Commit message: Add joint damping to all arm revolute joints to prevent gravity collapse
Arm joints had no damping/friction, causing them to fall freely under
gravity at startup (before JointPositionController receives first cmd).
This pushed the robot off its spawn position. Adding damping=10.0 and
friction=5.0 to joints 1-5 simulates real servo resistance.

Co-Authored-By: Claude Opus 4.6 <noreply@anthropic.com>

File: urdf/jetrover_description/urdf/arm.urdf.xacro (robot description, xacro)
@@ -140,4 +140,5 @@
       effort="1000"
       velocity="10" />
+    <dynamics damping="10.0" friction="5.0"/>
   </joint>
   <link
@@ -194,4 +195,5 @@
       effort="1000"
       velocity="10" />
+    <dynamics damping="10.0" friction="5.0"/>
   </joint>
   <link
@@ -248,4 +250,5 @@
       effort="1000"
       velocity="10" />
+    <dynamics damping="10.0" friction="5.0"/>
   </joint>
   <link
@@ -351,4 +354,5 @@
       effort="1000"
       velocity="10" />
+    <dynamics damping="10.0" friction="5.0"/>
   </joint>
   <link

File: urdf/jetrover_description/urdf/connect.urdf.xacro (robot description, xacro)
@@ -19,4 +19,5 @@
       effort="1000"
       velocity="10" />
+    <dynamics damping="10.0" friction="5.0"/>
   </joint>
 </robot>
