Commit message: Reduce joint damping to 2.0, remove PID I gain to fix arm instability
- Damping 10.0→2.0: still prevents gravity collapse but doesn't
  overwhelm PID control budget
- Friction 5.0→1.0: less resistance to commanded motion
- I gain→0: prevents integral windup that caused joint1 spinning
- cmd_max=50 (adequate for damping=2.0 joints)

File: urdf/jetrover_description/urdf/arm.urdf.xacro (robot description, xacro)
@@ -140,5 +140,5 @@
       effort="1000"
       velocity="10" />
-    <dynamics damping="10.0" friction="5.0"/>
+    <dynamics damping="2.0" friction="1.0"/>
   </joint>
   <link
@@ -195,5 +195,5 @@
       effort="1000"
       velocity="10" />
-    <dynamics damping="10.0" friction="5.0"/>
+    <dynamics damping="2.0" friction="1.0"/>
   </joint>
   <link
@@ -250,5 +250,5 @@
       effort="1000"
       velocity="10" />
-    <dynamics damping="10.0" friction="5.0"/>
+    <dynamics damping="2.0" friction="1.0"/>
   </joint>
   <link
@@ -354,5 +354,5 @@
       effort="1000"
       velocity="10" />
-    <dynamics damping="10.0" friction="5.0"/>
+    <dynamics damping="2.0" friction="1.0"/>
   </joint>
   <link

File: urdf/jetrover_description/urdf/connect.urdf.xacro (robot description, xacro)
@@ -19,5 +19,5 @@
       effort="1000"
       velocity="10" />
-    <dynamics damping="10.0" friction="5.0"/>
+    <dynamics damping="2.0" friction="1.0"/>
   </joint>
 </robot>

File: urdf/robot.urdf.xacro (robot description, xacro)
@@ -73,6 +73,6 @@
     </gazebo>
     <!-- ==================== Arm Joint Controllers ==================== -->
-    <!-- PID controllers for arm joints. cmd_max must exceed damping*velocity
-         to allow the controller to overcome joint damping during motion. -->
+    <!-- PID controllers for arm joints. Damping reduced to 2.0 so these
+         moderate gains can easily control the joints. No I gain to avoid windup. -->
     <gazebo>
         <plugin filename="gz-sim-joint-position-controller-system"
@@ -80,9 +80,9 @@
             <joint_name>joint1</joint_name>
             <topic>arm/joint1/cmd_pos</topic>
-            <p_gain>500</p_gain>
-            <i_gain>10</i_gain>
-            <d_gain>50</d_gain>
-            <cmd_max>100</cmd_max>
-            <cmd_min>-100</cmd_min>
+            <p_gain>200</p_gain>
+            <i_gain>0</i_gain>
+            <d_gain>20</d_gain>
+            <cmd_max>50</cmd_max>
+            <cmd_min>-50</cmd_min>
         </plugin>
     </gazebo>
@@ -92,9 +92,9 @@
             <joint_name>joint2</joint_name>
             <topic>arm/joint2/cmd_pos</topic>
-            <p_gain>500</p_gain>
-            <i_gain>10</i_gain>
-            <d_gain>50</d_gain>
-            <cmd_max>100</cmd_max>
-            <cmd_min>-100</cmd_min>
+            <p_gain>200</p_gain>
+            <i_gain>0</i_gain>
+            <d_gain>20</d_gain>
+            <cmd_max>50</cmd_max>
+            <cmd_min>-50</cmd_min>
         </plugin>
     </gazebo>
@@ -104,9 +104,9 @@
             <joint_name>joint3</joint_name>
             <topic>arm/joint3/cmd_pos</topic>
-            <p_gain>500</p_gain>
-            <i_gain>10</i_gain>
-            <d_gain>50</d_gain>
-            <cmd_max>100</cmd_max>
-            <cmd_min>-100</cmd_min>
+            <p_gain>200</p_gain>
+            <i_gain>0</i_gain>
+            <d_gain>20</d_gain>
+            <cmd_max>50</cmd_max>
+            <cmd_min>-50</cmd_min>
         </plugin>
     </gazebo>
@@ -116,9 +116,9 @@
             <joint_name>joint4</joint_name>
             <topic>arm/joint4/cmd_pos</topic>
-            <p_gain>500</p_gain>
-            <i_gain>10</i_gain>
-            <d_gain>50</d_gain>
-            <cmd_max>100</cmd_max>
-            <cmd_min>-100</cmd_min>
+            <p_gain>200</p_gain>
+            <i_gain>0</i_gain>
+            <d_gain>20</d_gain>
+            <cmd_max>50</cmd_max>
+            <cmd_min>-50</cmd_min>
         </plugin>
     </gazebo>
@@ -128,23 +128,23 @@
             <joint_name>joint5</joint_name>
             <topic>arm/joint5/cmd_pos</topic>
-            <p_gain>200</p_gain>
-            <i_gain>5</i_gain>
-            <d_gain>20</d_gain>
-            <cmd_max>50</cmd_max>
-            <cmd_min>-50</cmd_min>
-        </plugin>
-    </gazebo>
-    <!-- ==================== Gripper Controller ==================== -->
-    <!-- Only r_joint is actuated; l_joint and all linkage joints mimic it -->
-    <gazebo>
-        <plugin filename="gz-sim-joint-position-controller-system"
-                name="gz::sim::systems::JointPositionController">
-            <joint_name>r_joint</joint_name>
-            <topic>arm/gripper/cmd_pos</topic>
             <p_gain>100</p_gain>
-            <i_gain>5</i_gain>
+            <i_gain>0</i_gain>
             <d_gain>10</d_gain>
             <cmd_max>20</cmd_max>
             <cmd_min>-20</cmd_min>
+        </plugin>
+    </gazebo>
+    <!-- ==================== Gripper Controller ==================== -->
+    <!-- Only r_joint is actuated; l_joint and all linkage joints mimic it -->
+    <gazebo>
+        <plugin filename="gz-sim-joint-position-controller-system"
+                name="gz::sim::systems::JointPositionController">
+            <joint_name>r_joint</joint_name>
+            <topic>arm/gripper/cmd_pos</topic>
+            <p_gain>50</p_gain>
+            <i_gain>0</i_gain>
+            <d_gain>5</d_gain>
+            <cmd_max>10</cmd_max>
+            <cmd_min>-10</cmd_min>
         </plugin>
     </gazebo>

Commit message: Tune arm PID/damping for stable startup: damping=5.0, p=150/d=30, init delay 0.5s
Previous iteration (damping=2.0) let the arm fall during the 2s startup delay,
causing oscillation when PID kicked in. Now: moderate damping provides passive
gravity resistance, faster init sends home command before arm drifts, and
higher D gain dampens any residual oscillation.

File: urdf/jetrover_description/urdf/arm.urdf.xacro (robot description, xacro)
@@ -140,5 +140,5 @@
       effort="1000"
       velocity="10" />
-    <dynamics damping="2.0" friction="1.0"/>
+    <dynamics damping="5.0" friction="2.0"/>
   </joint>
   <link
@@ -195,5 +195,5 @@
       effort="1000"
       velocity="10" />
-    <dynamics damping="2.0" friction="1.0"/>
+    <dynamics damping="5.0" friction="2.0"/>
   </joint>
   <link
@@ -250,5 +250,5 @@
       effort="1000"
       velocity="10" />
-    <dynamics damping="2.0" friction="1.0"/>
+    <dynamics damping="5.0" friction="2.0"/>
   </joint>
   <link
@@ -354,5 +354,5 @@
       effort="1000"
       velocity="10" />
-    <dynamics damping="2.0" friction="1.0"/>
+    <dynamics damping="5.0" friction="2.0"/>
   </joint>
   <link

File: urdf/jetrover_description/urdf/connect.urdf.xacro (robot description, xacro)
@@ -19,5 +19,5 @@
       effort="1000"
       velocity="10" />
-    <dynamics damping="2.0" friction="1.0"/>
+    <dynamics damping="5.0" friction="2.0"/>
   </joint>
 </robot>

File: urdf/robot.urdf.xacro (robot description, xacro)
@@ -73,6 +73,6 @@
     </gazebo>
     <!-- ==================== Arm Joint Controllers ==================== -->
-    <!-- PID controllers for arm joints. Damping reduced to 2.0 so these
-         moderate gains can easily control the joints. No I gain to avoid windup. -->
+    <!-- PID controllers for arm joints. Damping=5.0 provides gravity resistance
+         while PID p=150/d=30 provides responsive control. No I gain to avoid windup. -->
     <gazebo>
         <plugin filename="gz-sim-joint-position-controller-system"
@@ -80,7 +80,7 @@
             <joint_name>joint1</joint_name>
             <topic>arm/joint1/cmd_pos</topic>
-            <p_gain>200</p_gain>
-            <i_gain>0</i_gain>
-            <d_gain>20</d_gain>
+            <p_gain>150</p_gain>
+            <i_gain>0</i_gain>
+            <d_gain>30</d_gain>
             <cmd_max>50</cmd_max>
             <cmd_min>-50</cmd_min>
@@ -92,7 +92,7 @@
             <joint_name>joint2</joint_name>
             <topic>arm/joint2/cmd_pos</topic>
-            <p_gain>200</p_gain>
-            <i_gain>0</i_gain>
-            <d_gain>20</d_gain>
+            <p_gain>150</p_gain>
+            <i_gain>0</i_gain>
+            <d_gain>30</d_gain>
             <cmd_max>50</cmd_max>
             <cmd_min>-50</cmd_min>
@@ -104,7 +104,7 @@
             <joint_name>joint3</joint_name>
             <topic>arm/joint3/cmd_pos</topic>
-            <p_gain>200</p_gain>
-            <i_gain>0</i_gain>
-            <d_gain>20</d_gain>
+            <p_gain>150</p_gain>
+            <i_gain>0</i_gain>
+            <d_gain>30</d_gain>
             <cmd_max>50</cmd_max>
             <cmd_min>-50</cmd_min>
@@ -116,7 +116,7 @@
             <joint_name>joint4</joint_name>
             <topic>arm/joint4/cmd_pos</topic>
-            <p_gain>200</p_gain>
-            <i_gain>0</i_gain>
-            <d_gain>20</d_gain>
+            <p_gain>150</p_gain>
+            <i_gain>0</i_gain>
+            <d_gain>30</d_gain>
             <cmd_max>50</cmd_max>
             <cmd_min>-50</cmd_min>
@@ -128,7 +128,7 @@
             <joint_name>joint5</joint_name>
             <topic>arm/joint5/cmd_pos</topic>
-            <p_gain>100</p_gain>
-            <i_gain>0</i_gain>
-            <d_gain>10</d_gain>
+            <p_gain>80</p_gain>
+            <i_gain>0</i_gain>
+            <d_gain>15</d_gain>
             <cmd_max>20</cmd_max>
             <cmd_min>-20</cmd_min>

Commit message: High damping (20.0) for overdamped arm stability, PID p=200/d=20/cmd_max=80
Low-inertia links (~1e-5 kg·m²) with moderate damping caused numerical
instability — tiny torques created enormous accelerations. Now using
damping=20 so max velocity = cmd_max/damping = 4 rad/s, making the
system inherently overdamped. Also added damping to gripper r_joint.

File: urdf/jetrover_description/urdf/arm.urdf.xacro (robot description, xacro)
@@ -140,5 +140,5 @@
       effort="1000"
       velocity="10" />
-    <dynamics damping="5.0" friction="2.0"/>
+    <dynamics damping="20.0" friction="5.0"/>
   </joint>
   <link
@@ -195,5 +195,5 @@
       effort="1000"
       velocity="10" />
-    <dynamics damping="5.0" friction="2.0"/>
+    <dynamics damping="20.0" friction="5.0"/>
   </joint>
   <link
@@ -250,5 +250,5 @@
       effort="1000"
       velocity="10" />
-    <dynamics damping="5.0" friction="2.0"/>
+    <dynamics damping="20.0" friction="5.0"/>
   </joint>
   <link
@@ -354,5 +354,5 @@
       effort="1000"
       velocity="10" />
-    <dynamics damping="5.0" friction="2.0"/>
+    <dynamics damping="20.0" friction="5.0"/>
   </joint>
   <link

File: urdf/jetrover_description/urdf/connect.urdf.xacro (robot description, xacro)
@@ -19,5 +19,5 @@
       effort="1000"
       velocity="10" />
-    <dynamics damping="5.0" friction="2.0"/>
+    <dynamics damping="20.0" friction="5.0"/>
   </joint>
 </robot>

File: urdf/jetrover_description/urdf/gripper.urdf.xacro (robot description, xacro)
@@ -55,4 +55,5 @@
       effort="1000"
       velocity="10" />
+    <dynamics damping="10.0" friction="2.0"/>
   </joint>
   <link

File: urdf/robot.urdf.xacro (robot description, xacro)
@@ -73,6 +73,7 @@
     </gazebo>
     <!-- ==================== Arm Joint Controllers ==================== -->
-    <!-- PID controllers for arm joints. Damping=5.0, low cmd_max to prevent
-         oscillation on these low-inertia links (~1e-5 kg·m²). No I gain. -->
+    <!-- PID controllers for arm joints. High damping=20 makes system overdamped,
+         preventing oscillation. P=200 + cmd_max=80 overcomes damping.
+         Max velocity = cmd_max/damping = 4 rad/s. No I gain to avoid windup. -->
     <gazebo>
         <plugin filename="gz-sim-joint-position-controller-system"
@@ -80,9 +81,9 @@
             <joint_name>joint1</joint_name>
             <topic>arm/joint1/cmd_pos</topic>
-            <p_gain>100</p_gain>
-            <i_gain>0</i_gain>
-            <d_gain>10</d_gain>
-            <cmd_max>20</cmd_max>
-            <cmd_min>-20</cmd_min>
+            <p_gain>200</p_gain>
+            <i_gain>0</i_gain>
+            <d_gain>20</d_gain>
+            <cmd_max>80</cmd_max>
+            <cmd_min>-80</cmd_min>
         </plugin>
     </gazebo>
@@ -92,9 +93,9 @@
             <joint_name>joint2</joint_name>
             <topic>arm/joint2/cmd_pos</topic>
-            <p_gain>100</p_gain>
-            <i_gain>0</i_gain>
-            <d_gain>10</d_gain>
-            <cmd_max>20</cmd_max>
-            <cmd_min>-20</cmd_min>
+            <p_gain>200</p_gain>
+            <i_gain>0</i_gain>
+            <d_gain>20</d_gain>
+            <cmd_max>80</cmd_max>
+            <cmd_min>-80</cmd_min>
         </plugin>
     </gazebo>
@@ -104,9 +105,9 @@
             <joint_name>joint3</joint_name>
             <topic>arm/joint3/cmd_pos</topic>
-            <p_gain>100</p_gain>
-            <i_gain>0</i_gain>
-            <d_gain>10</d_gain>
-            <cmd_max>20</cmd_max>
-            <cmd_min>-20</cmd_min>
+            <p_gain>200</p_gain>
+            <i_gain>0</i_gain>
+            <d_gain>20</d_gain>
+            <cmd_max>80</cmd_max>
+            <cmd_min>-80</cmd_min>
         </plugin>
     </gazebo>
@@ -116,9 +117,9 @@
             <joint_name>joint4</joint_name>
             <topic>arm/joint4/cmd_pos</topic>
-            <p_gain>100</p_gain>
-            <i_gain>0</i_gain>
-            <d_gain>10</d_gain>
-            <cmd_max>20</cmd_max>
-            <cmd_min>-20</cmd_min>
+            <p_gain>200</p_gain>
+            <i_gain>0</i_gain>
+            <d_gain>20</d_gain>
+            <cmd_max>80</cmd_max>
+            <cmd_min>-80</cmd_min>
         </plugin>
     </gazebo>
@@ -128,9 +129,9 @@
             <joint_name>joint5</joint_name>
             <topic>arm/joint5/cmd_pos</topic>
-            <p_gain>50</p_gain>
-            <i_gain>0</i_gain>
-            <d_gain>5</d_gain>
-            <cmd_max>10</cmd_max>
-            <cmd_min>-10</cmd_min>
+            <p_gain>100</p_gain>
+            <i_gain>0</i_gain>
+            <d_gain>10</d_gain>
+            <cmd_max>40</cmd_max>
+            <cmd_min>-40</cmd_min>
         </plugin>
     </gazebo>

Commit message: Damping=10, cmd_max=40: compromise between stability and joint3/4 response
Damping=20 prevented joints 3/4 from moving entirely despite PID commands
being received on Gazebo side. Damping=10 provides moderate damping while
allowing all joints to respond to position commands.

File: urdf/jetrover_description/urdf/arm.urdf.xacro (robot description, xacro)
@@ -140,5 +140,5 @@
       effort="1000"
       velocity="10" />
-    <dynamics damping="20.0" friction="5.0"/>
+    <dynamics damping="10.0" friction="2.0"/>
   </joint>
   <link
@@ -195,5 +195,5 @@
       effort="1000"
       velocity="10" />
-    <dynamics damping="20.0" friction="5.0"/>
+    <dynamics damping="10.0" friction="2.0"/>
   </joint>
   <link
@@ -250,5 +250,5 @@
       effort="1000"
       velocity="10" />
-    <dynamics damping="20.0" friction="5.0"/>
+    <dynamics damping="10.0" friction="2.0"/>
   </joint>
   <link
@@ -354,5 +354,5 @@
       effort="1000"
       velocity="10" />
-    <dynamics damping="20.0" friction="5.0"/>
+    <dynamics damping="10.0" friction="2.0"/>
   </joint>
   <link

File: urdf/jetrover_description/urdf/connect.urdf.xacro (robot description, xacro)
@@ -19,5 +19,5 @@
       effort="1000"
       velocity="10" />
-    <dynamics damping="20.0" friction="5.0"/>
+    <dynamics damping="10.0" friction="2.0"/>
   </joint>
 </robot>

File: urdf/robot.urdf.xacro (robot description, xacro)
@@ -73,7 +73,6 @@
     </gazebo>
     <!-- ==================== Arm Joint Controllers ==================== -->
-    <!-- PID controllers for arm joints. High damping=20 makes system overdamped,
-         preventing oscillation. P=200 + cmd_max=80 overcomes damping.
-         Max velocity = cmd_max/damping = 4 rad/s. No I gain to avoid windup. -->
+    <!-- PID controllers for arm joints. Damping=10 balances stability with
+         responsiveness. Max velocity = cmd_max/damping = 4 rad/s. -->
     <gazebo>
         <plugin filename="gz-sim-joint-position-controller-system"
@@ -84,6 +83,6 @@
             <i_gain>0</i_gain>
             <d_gain>20</d_gain>
-            <cmd_max>80</cmd_max>
-            <cmd_min>-80</cmd_min>
+            <cmd_max>40</cmd_max>
+            <cmd_min>-40</cmd_min>
         </plugin>
     </gazebo>
@@ -96,6 +95,6 @@
             <i_gain>0</i_gain>
             <d_gain>20</d_gain>
-            <cmd_max>80</cmd_max>
-            <cmd_min>-80</cmd_min>
+            <cmd_max>40</cmd_max>
+            <cmd_min>-40</cmd_min>
         </plugin>
     </gazebo>
@@ -108,6 +107,6 @@
             <i_gain>0</i_gain>
             <d_gain>20</d_gain>
-            <cmd_max>80</cmd_max>
-            <cmd_min>-80</cmd_min>
+            <cmd_max>40</cmd_max>
+            <cmd_min>-40</cmd_min>
         </plugin>
     </gazebo>
@@ -120,6 +119,6 @@
             <i_gain>0</i_gain>
             <d_gain>20</d_gain>
-            <cmd_max>80</cmd_max>
-            <cmd_min>-80</cmd_min>
+            <cmd_max>40</cmd_max>
+            <cmd_min>-40</cmd_min>
         </plugin>
     </gazebo>
@@ -132,6 +131,6 @@
             <i_gain>0</i_gain>
             <d_gain>10</d_gain>
-            <cmd_max>40</cmd_max>
-            <cmd_min>-40</cmd_min>
+            <cmd_max>20</cmd_max>
+            <cmd_min>-20</cmd_min>
         </plugin>
     </gazebo>

Commit message: Revert plugin names, remove link4/servo_link2 collisions to test joint4
Plugin name MUST be the system class name (gz::sim::systems::*), not arbitrary.
Removing link4 and servo_link2 collision meshes to test if self-collision
is preventing joint4 from moving.

File: urdf/jetrover_description/urdf/arm.urdf.xacro (robot description, xacro)
@@ -223,13 +223,4 @@
       <material name="green"/>
     </visual>
-    <collision>
-      <origin
-        xyz="0 0 0"
-        rpy="0 0 0" />
-      <geometry>
-        <mesh
-          filename="package://jetrover_description/meshes/arm/link4_collision.stl" />
-      </geometry>
-    </collision>
   </link>
   <joint
@@ -278,13 +269,4 @@
       <material name="black"/>
     </visual>
-    <collision>
-      <origin
-        xyz="0 0 0"
-        rpy="0 0 0" />
-      <geometry>
-        <mesh
-          filename="package://jetrover_description/meshes/arm/servo_link2_collision.stl" />
-      </geometry>
-    </collision>
   </link>
   <joint

File: urdf/robot.urdf.xacro (robot description, xacro)
@@ -78,5 +78,5 @@
     <gazebo>
         <plugin filename="gz-sim-joint-position-controller-system"
-                name="joint1_position_controller">
+                name="gz::sim::systems::JointPositionController">
             <joint_name>joint1</joint_name>
             <topic>arm/joint1/cmd_pos</topic>
@@ -90,5 +90,5 @@
     <gazebo>
         <plugin filename="gz-sim-joint-position-controller-system"
-                name="joint2_position_controller">
+                name="gz::sim::systems::JointPositionController">
             <joint_name>joint2</joint_name>
             <topic>arm/joint2/cmd_pos</topic>
@@ -102,5 +102,5 @@
     <gazebo>
         <plugin filename="gz-sim-joint-position-controller-system"
-                name="joint3_position_controller">
+                name="gz::sim::systems::JointPositionController">
             <joint_name>joint3</joint_name>
             <topic>arm/joint3/cmd_pos</topic>
@@ -114,5 +114,5 @@
     <gazebo>
         <plugin filename="gz-sim-joint-position-controller-system"
-                name="joint4_position_controller">
+                name="gz::sim::systems::JointPositionController">
             <joint_name>joint4</joint_name>
             <topic>arm/joint4/cmd_pos</topic>
@@ -126,5 +126,5 @@
     <gazebo>
         <plugin filename="gz-sim-joint-position-controller-system"
-                name="joint5_position_controller">
+                name="gz::sim::systems::JointPositionController">
             <joint_name>joint5</joint_name>
             <topic>arm/joint5/cmd_pos</topic>
@@ -140,5 +140,5 @@
     <gazebo>
         <plugin filename="gz-sim-joint-position-controller-system"
-                name="gripper_position_controller">
+                name="gz::sim::systems::JointPositionController">
             <joint_name>r_joint</joint_name>
             <topic>arm/gripper/cmd_pos</topic>

Commit message: Lower damping to 1.0 and cmd_max to 5 for joints 4/5 (low-inertia fix)
Extreme damping/inertia ratio (~100k) likely causes DART numerical issues.
Joint4 inertia is ~0.0001 with damping=10 → impossible to move. Reducing
damping to 1.0 and cmd_max to 5 for a manageable ratio of ~10k.

File: urdf/jetrover_description/urdf/arm.urdf.xacro (robot description, xacro)
@@ -241,5 +241,5 @@
       effort="1000"
       velocity="10" />
-    <dynamics damping="10.0" friction="2.0"/>
+    <dynamics damping="1.0" friction="0.5"/>
   </joint>
   <link
@@ -336,5 +336,5 @@
       effort="1000"
       velocity="10" />
-    <dynamics damping="10.0" friction="2.0"/>
+    <dynamics damping="1.0" friction="0.5"/>
   </joint>
   <link

File: urdf/robot.urdf.xacro (robot description, xacro)
@@ -117,9 +117,9 @@
             <joint_name>joint4</joint_name>
             <topic>arm/joint4/cmd_pos</topic>
-            <p_gain>200</p_gain>
-            <i_gain>0</i_gain>
-            <d_gain>0</d_gain>
-            <cmd_max>40</cmd_max>
-            <cmd_min>-40</cmd_min>
+            <p_gain>50</p_gain>
+            <i_gain>0</i_gain>
+            <d_gain>0</d_gain>
+            <cmd_max>5</cmd_max>
+            <cmd_min>-5</cmd_min>
         </plugin>
     </gazebo>
@@ -129,9 +129,9 @@
             <joint_name>joint5</joint_name>
             <topic>arm/joint5/cmd_pos</topic>
-            <p_gain>100</p_gain>
-            <i_gain>0</i_gain>
-            <d_gain>0</d_gain>
-            <cmd_max>20</cmd_max>
-            <cmd_min>-20</cmd_min>
+            <p_gain>50</p_gain>
+            <i_gain>0</i_gain>
+            <d_gain>0</d_gain>
+            <cmd_max>5</cmd_max>
+            <cmd_min>-5</cmd_min>
         </plugin>
     </gazebo>

Commit message: Apply damping=1.0, cmd_max=5 to joint3 as well (same inertia ratio fix)

File: urdf/jetrover_description/urdf/arm.urdf.xacro (robot description, xacro)
@@ -195,5 +195,5 @@
       effort="1000"
       velocity="10" />
-    <dynamics damping="10.0" friction="2.0"/>
+    <dynamics damping="1.0" friction="0.5"/>
   </joint>
   <link

File: urdf/robot.urdf.xacro (robot description, xacro)
@@ -105,9 +105,9 @@
             <joint_name>joint3</joint_name>
             <topic>arm/joint3/cmd_pos</topic>
-            <p_gain>200</p_gain>
-            <i_gain>0</i_gain>
-            <d_gain>0</d_gain>
-            <cmd_max>40</cmd_max>
-            <cmd_min>-40</cmd_min>
+            <p_gain>50</p_gain>
+            <i_gain>0</i_gain>
+            <d_gain>0</d_gain>
+            <cmd_max>5</cmd_max>
+            <cmd_min>-5</cmd_min>
         </plugin>
     </gazebo>
