Commit message: Remove depth camera collision meshes to test joint4 self-collision hypothesis
Joint4 refuses to move despite receiving commands — suspecting collision
between camera_connect_link/depth_cam_link meshes (merged with link4 via
fixed joints) and link3. Removing collisions to verify.

File: urdf/jetrover_description/urdf/depth_camera.urdf.xacro (robot description, xacro)
@@ -28,13 +28,4 @@
       <material name="black"/>
     </visual>
-    <collision>
-      <origin
-        xyz="0 0 0"
-        rpy="0 0 0" />
-      <geometry>
-        <mesh
-          filename="package://jetrover_description/meshes/arm/camera_connect_link.STL" />
-      </geometry>
-    </collision>
   </link>
   <joint
@@ -81,13 +72,4 @@
       </material>
     </visual>
-    <collision>
-      <origin
-        xyz="0 0 0"
-        rpy="0 0 0" />
-      <geometry>
-        <mesh
-          filename="package://jetrover_description/meshes/arm/depth_cam_link_collision.stl" />
-      </geometry>
-    </collision>
   </link>
   <joint
