Commit message: Fix gripper: lower damping, add dynamics to mimic joints, tune PID
- r_joint: damping 10.0 -> 0.5, friction 2.0 -> 0.1
- All mimic joints: add damping=0.1, friction=0.05
- Gripper PID: P=100, I=30, i_max=±5 (was P=50, I=0)
- High damping on tiny-inertia gripper joints caused same issue as arm

Co-Authored-By: Claude Opus 4.6 <noreply@anthropic.com>

File: urdf/jetrover_description/urdf/gripper.urdf.xacro (robot description, xacro)
@@ -55,5 +55,5 @@
       effort="1000"
       velocity="10" />
-    <dynamics damping="10.0" friction="2.0"/>
+    <dynamics damping="0.5" friction="0.1"/>
   </joint>
   <link
@@ -110,4 +110,5 @@
       effort="1000"
       velocity="10" />
+    <dynamics damping="0.1" friction="0.05"/>
     <mimic
       joint="r_joint"
@@ -168,4 +169,5 @@
       effort="1000"
       velocity="10" />
+    <dynamics damping="0.1" friction="0.05"/>
     <mimic
       joint="r_joint"
@@ -226,4 +228,5 @@
       effort="1000"
       velocity="10" />
+    <dynamics damping="0.1" friction="0.05"/>
     <mimic
       joint="r_joint"
@@ -284,4 +287,5 @@
       effort="1000"
       velocity="10" />
+    <dynamics damping="0.1" friction="0.05"/>
     <mimic
       joint="r_joint"
@@ -342,4 +346,5 @@
       effort="1000"
       velocity="10" />
+    <dynamics damping="0.1" friction="0.05"/>
     <mimic
       joint="r_joint"

File: urdf/robot.urdf.xacro (robot description, xacro)
@@ -154,7 +154,9 @@
             <joint_name>r_joint</joint_name>
             <topic>arm/gripper/cmd_pos</topic>
-            <p_gain>50</p_gain>
-            <i_gain>0</i_gain>
-            <d_gain>0</d_gain>
+            <p_gain>100</p_gain>
+            <i_gain>30</i_gain>
+            <d_gain>0</d_gain>
+            <i_max>5</i_max>
+            <i_min>-5</i_min>
             <cmd_max>10</cmd_max>
             <cmd_min>-10</cmd_min>

Commit message: Lower gripper damping further to fix DART numerical issue
- r_joint and all mimic joints: damping=0.001, friction=0.001
- Previous damping=0.5 still too high for ~4e-7 kg*m^2 inertia
- Damping/inertia ratio must be reasonable for DART solver

Co-Authored-By: Claude Opus 4.6 <noreply@anthropic.com>

File: urdf/jetrover_description/urdf/gripper.urdf.xacro (robot description, xacro)
@@ -55,5 +55,5 @@
       effort="1000"
       velocity="10" />
-    <dynamics damping="0.5" friction="0.1"/>
+    <dynamics damping="0.001" friction="0.001"/>
   </joint>
   <link
@@ -110,5 +110,5 @@
       effort="1000"
       velocity="10" />
-    <dynamics damping="0.1" friction="0.05"/>
+    <dynamics damping="0.001" friction="0.001"/>
     <mimic
       joint="r_joint"
@@ -169,5 +169,5 @@
       effort="1000"
       velocity="10" />
-    <dynamics damping="0.1" friction="0.05"/>
+    <dynamics damping="0.001" friction="0.001"/>
     <mimic
       joint="r_joint"
@@ -228,5 +228,5 @@
       effort="1000"
       velocity="10" />
-    <dynamics damping="0.1" friction="0.05"/>
+    <dynamics damping="0.001" friction="0.001"/>
     <mimic
       joint="r_joint"
@@ -287,5 +287,5 @@
       effort="1000"
       velocity="10" />
-    <dynamics damping="0.1" friction="0.05"/>
+    <dynamics damping="0.001" friction="0.001"/>
     <mimic
       joint="r_joint"
@@ -346,5 +346,5 @@
       effort="1000"
       velocity="10" />
-    <dynamics damping="0.1" friction="0.05"/>
+    <dynamics damping="0.001" friction="0.001"/>
     <mimic
       joint="r_joint"
