Commit message: Add fixed body camera for room scanning perception
- Add body_cam_link on front of base_link, tilted 30deg down
- body_cam_optical_frame with standard optical convention
- Body camera publishes on /camera/* topics (for perception node)
- Arm camera moved to /arm_camera/* topics (for pick/place later)
- Body camera eliminates arm stability issues for perception testing

File: urdf/robot.urdf.xacro (robot description, xacro)
@@ -13,4 +13,25 @@
     <xacro:include filename="$(find llm_robot_task_planner)/urdf/jetrover_description/urdf/arm.urdf.xacro"/>
     <xacro:include filename="$(find llm_robot_task_planner)/urdf/jetrover_description/urdf/gripper.urdf.xacro"/>
+    <!-- ==================== Fixed Body Camera (for perception scanning) ==================== -->
+    <!-- Front-facing RGBD camera on robot body, tilted 30° down to see floor/cubes -->
+    <link name="body_cam_link">
+        <inertial>
+            <mass value="0.01"/>
+            <inertia ixx="1e-6" ixy="0" ixz="0" iyy="1e-6" iyz="0" izz="1e-6"/>
+        </inertial>
+    </link>
+    <joint name="body_cam_joint" type="fixed">
+        <!-- Mounted at front-top of base_link, tilted 30° down (pitch = 0.52 rad) -->
+        <origin xyz="0.12 0.0 0.06" rpy="0 0.52 0"/>
+        <parent link="base_link"/>
+        <child link="body_cam_link"/>
+    </joint>
+    <!-- Optical frame (standard: z-forward, x-right, y-down) -->
+    <link name="body_cam_optical_frame"/>
+    <joint name="body_cam_optical_joint" type="fixed">
+        <origin xyz="0 0 0" rpy="-1.5708 0 -1.5708"/>
+        <parent link="body_cam_link"/>
+        <child link="body_cam_optical_frame"/>
+    </joint>
     <!-- ==================== Gazebo Plugins ==================== -->
     <!-- Diff drive (simpler than mecanum for initial testing, upgrade later) -->
@@ -167,9 +188,9 @@
         </sensor>
     </gazebo>
-    <!-- RGBD camera on depth_cam_frame (arm-mounted, matches Astra Pro specs) -->
-    <gazebo reference="depth_cam_frame">
-        <sensor name="rgbd_camera" type="rgbd_camera">
+    <!-- Fixed body RGBD camera for room scanning / perception -->
+    <gazebo reference="body_cam_optical_frame">
+        <sensor name="body_rgbd_camera" type="rgbd_camera">
             <topic>camera</topic>
-            <gz_frame_id>depth_cam_frame</gz_frame_id>
+            <gz_frame_id>body_cam_optical_frame</gz_frame_id>
             <update_rate>15</update_rate>
             <always_on>true</always_on>
@@ -194,3 +215,30 @@
         </sensor>
     </gazebo>
+    <!-- Arm-mounted RGBD camera (for pick/place guidance, DC5) -->
+    <gazebo reference="depth_cam_frame">
+        <sensor name="arm_rgbd_camera" type="rgbd_camera">
+            <topic>arm_camera</topic>
+            <gz_frame_id>depth_cam_frame</gz_frame_id>
+            <update_rate>15</update_rate>
+            <always_on>true</always_on>
+            <camera>
+                <horizontal_fov>1.047</horizontal_fov>
+                <image>
+                    <width>640</width>
+                    <height>480</height>
+                    <format>R8G8B8</format>
+                </image>
+                <clip>
+                    <near>0.1</near>
+                    <far>10.0</far>
+                </clip>
+                <depth_camera>
+                    <clip>
+                        <near>0.1</near>
+                        <far>10.0</far>
+                    </clip>
+                </depth_camera>
+            </camera>
+        </sensor>
+    </gazebo>
 </robot>

Commit message: Increase cube size to 5cm (PRD spec) and adjust camera for detection
- Cubes: 3cm -> 5cm (matches PRD 5-8cm spec, visible at room distances)
- Body camera tilt: 30deg -> 15deg (sees further ahead, covers more floor)
- MIN_CONTOUR_AREA: 100 -> 30 (detect smaller objects in frame)
- Updated cube z-positions and inertia for new size

File: urdf/robot.urdf.xacro (robot description, xacro)
@@ -22,6 +22,6 @@
     </link>
     <joint name="body_cam_joint" type="fixed">
-        <!-- Mounted at front-top of base_link, tilted 30° down (pitch = 0.52 rad) -->
-        <origin xyz="0.12 0.0 0.06" rpy="0 0.52 0"/>
+        <!-- Mounted at front-top of base_link, tilted 15° down (pitch = 0.26 rad) -->
+        <origin xyz="0.12 0.0 0.06" rpy="0 0.26 0"/>
         <parent link="base_link"/>
         <child link="body_cam_link"/>

Commit message: Widen body camera FOV to 90deg and increase tilt to 20deg

File: urdf/robot.urdf.xacro (robot description, xacro)
@@ -22,6 +22,6 @@
     </link>
     <joint name="body_cam_joint" type="fixed">
-        <!-- Mounted at front-top of base_link, tilted 15° down (pitch = 0.26 rad) -->
-        <origin xyz="0.12 0.0 0.06" rpy="0 0.26 0"/>
+        <!-- Mounted at front-top of base_link, tilted 20° down (pitch = 0.35 rad) -->
+        <origin xyz="0.12 0.0 0.06" rpy="0 0.35 0"/>
         <parent link="base_link"/>
         <child link="body_cam_link"/>
@@ -197,5 +197,5 @@
             <always_on>true</always_on>
             <camera>
-                <horizontal_fov>1.047</horizontal_fov>
+                <horizontal_fov>1.57</horizontal_fov>
                 <image>
                     <width>640</width>
@@ -204,10 +204,10 @@
                 </image>
                 <clip>
-                    <near>0.1</near>
+                    <near>0.05</near>
                     <far>10.0</far>
                 </clip>
                 <depth_camera>
                     <clip>
-                        <near>0.1</near>
+                        <near>0.05</near>
                         <far>10.0</far>
                     </clip>
